File: schematic.sch (KiCad schematic (older format))
At the start: 20 parts, among them T1 MCP4725A1T-E/CH, T2 MCP4725A1T-E/CH, U01 VDD, U010 VDD, U03 VDD, U05 VDD, U07 VDD, U08 GND, U2 10K, U4 10K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

Commit message: Remove stray node
Connections:
- wire segments 57 -> 56
Changed lines of the file:
@@
 	1550 1600 1550 2400
-Wire Wire Line
-	1650 1700 1650 1800
 Wire Wire Line
 	5050 2400 1550 2400
@@
 	-1   0    0    1
 $EndComp
-Connection ~ 1650 1800
 Wire Wire Line
-	1650 1800 1650 2500
+	1650 1700 1650 2500
 $EndSCHEMATC
